File: hardware/static_relay/static_relay.sch (KiCad schematic (older format))
At the start: 6 parts, among them IC1 MOC3022M, P1 CONN_2, P2 CONN_1, P3 CONN_1, U1 TRIAC

Commit message: hardware update
Connections:
- wire segments 12 -> 11
Other:
- moved on the sheet: IC1, P1, P2, P3, R1, U1
Changed lines of the file:
@@
-EESchema Schematic File Version 2  date dim. 19 mai 2013 22:09:36 CEST
+EESchema Schematic File Version 2
 LIBS:power
 LIBS:device
@@
 LIBS:contrib
 LIBS:valves
+LIBS:Conn-raspberry
 LIBS:static_relay-cache
-LIBS:pwr_lampe-cache
 EELAYER 24 0
 EELAYER END
@@
 Sheet 1 1
 Title "static relay"
-Date "19 may 2013"
+Date "20 may 2013"
 Rev "1"
 Comp "JbLb for Haum"
@@
 L TRIAC U1
 U 1 1 51992C6F
-P 4500 2150
-F 0 "U1" H 4250 2500 70  0000 C CNN
-F 1 "TRIAC" H 4200 1900 60  0000 C CNN
-F 2 "" H 4500 2150 60  0001 C CNN
-F 3 "" H 4500 2150 60  0001 C CNN
-	1    4500 2150
+P 10000 2450
+F 0 "U1" H 9750 2800 70  0000 C CNN
+F 1 "TRIAC" H 9700 2200 60  0000 C CNN
+F 2 "" H 10000 2450 60  0001 C CNN
+F 3 "" H 10000 2450 60  0001 C CNN
+	1    10000 2450
 	1    0    0    -1
 $EndComp
@@
 L R R1
 U 1 1 51992C75
-P 3500 1750
-F 0 "R1" V 3580 1750 50  0000 C CNN
-F 1 "470" V 3500 1750 50  0000 C CNN
-F 2 "" H 3500 1750 60  0001 C CNN
-F 3 "" H 3500 1750 60  0001 C CNN
-	1    3500 1750
+P 9000 2050
+F 0 "R1" V 9080 2050 50  0000 C CNN
+F 1 "470" V 9000 2050 50  0000 C CNN
+F 2 "" H 9000 2050 60  0001 C CNN
+F 3 "" H 9000 2050 60  0001 C CNN
+	1    9000 2050
 	0    1    1    0
 $EndComp
@@
 L MOC3022M IC1
 U 1 1 51992C78
-P 2750 2250
-F 0 "IC1" H 2536 2429 40  0000 C CNN
-F 1 "MOC3022M" H 2850 2065 40  0000 C CNN
-F 2 "DIP6" H 2586 2075 29  0000 C CNN
-F 3 "" H 2750 2250 60  0001 C CNN
-	1    2750 2250
+P 8250 2550
+F 0 "IC1" H 8036 2729 40  0000 C CNN
+F 1 "MOC3022M" H 8350 2365 40  0000 C CNN
+F 2 "DIP6" H 8086 2375 29  0000 C CNN
+F 3 "" H 8250 2550 60  0001 C CNN
+	1    8250 2550
 	1    0    0    -1
 $EndComp
-Wire Wire Line
-	4300 4550 4300 3950
 $Comp
 L CONN_2 P1
 U 1 1 51992D60
-P 1950 2250
-F 0 "P1" V 1900 2250 40  0000 C CNN
-F 1 "CONN_2" V 2000 2250 40  0000 C CNN
-F 2 "" H 1950 2250 60  0001 C CNN
-F 3 "" H 1950 2250 60  0001 C CNN
-	1    1950 2250
+P 7450 2550
+F 0 "P1" V 7400 2550 40  0000 C CNN
+F 1 "CONN_2" V 7500 2550 40  0000 C CNN
+F 2 "" H 7450 2550 60  0001 C CNN
+F 3 "" H 7450 2550 60  0001 C CNN
+	1    7450 2550
 	-1   0    0    -1
 $EndComp
@@
 L CONN_1 P2
 U 1 1 51992D72
-P 2000 1000
-F 0 "P2" H 2080 1000 40  0000 L CNN
-F 1 "CONN_1" H 2000 1055 30  0001 C CNN
-F 2 "~" H 2000 1000 60  0000 C CNN
-F 3 "~" H 2000 1000 60  0000 C CNN
-	1    2000 1000
+P 7500 1300
+F 0 "P2" H 7580 1300 40  0000 L CNN
+F 1 "CONN_1" H 7500 1355 30  0001 C CNN
+F 2 "~" H 7500 1300 60  0000 C CNN
+F 3 "~" H 7500 1300 60  0000 C CNN
+	1    7500 1300
 	-1   0    0    1
 $EndComp
@@
 L CONN_1 P3
 U 1 1 51992D81
-P 2000 1250
-F 0 "P3" H 2080 1250 40  0000 L CNN
-F 1 "CONN_1" H 2000 1305 30  0001 C CNN
-F 2 "~" H 2000 1250 60  0000 C CNN
-F 3 "~" H 2000 1250 60  0000 C CNN
-	1    2000 1250
+P 7500 1550
+F 0 "P3" H 7580 1550 40  0000 L CNN
+F 1 "CONN_1" H 7500 1605 30  0001 C CNN
+F 2 "~" H 7500 1550 60  0000 C CNN
+F 3 "~" H 7500 1550 60  0000 C CNN
+	1    7500 1550
 	-1   0    0    1
 $EndComp
 Wire Wire Line
-	4000 2350 3100 2350
+	9500 2650 8600 2650
 Wire Wire Line
-	4500 1750 3750 1750
+	10000 2050 9250 2050
 Wire Wire Line
-	3250 1750 3100 1750
+	8750 2050 8600 2050
 Wire Wire Line
-	3100 1750 3100 2150
+	8600 2050 8600 2450
 Wire Wire Line
-	2150 1250 4500 1250
+	7650 1550 10000 1550
 Wire Wire Line
-	4500 1250 4500 1750
+	10000 1550 10000 2050
 Wire Wire Line
-	2150 1000 4900 1000
+	7650 1300 10400 1300
 Wire Wire Line
-	4900 1000 4900 2400
+	10400 1300 10400 2700
 Wire Wire Line
-	4900 2400 4500 2400
+	10400 2700 10000 2700
 Wire Wire Line
-	2300 2150 2400 2150
+	7800 2450 7900 2450
 Wire Wire Line
-	2400 2350 2300 2350
+	7900 2650 7800 2650
 $EndSCHEMATC
